Commit message: changed joint default pos in URDF, updated sim params

File: my-robot/robot.urdf (robot description, URDF)
Before this commit: robot onshape, 2 links, 1 joints
Joints:
- joint hip: origin xyz=-0.020822569739601552719 0.01393648576781737064 -0.016207791599192972187 rpy=-1.570796326794896558 0.39827133476487169839 1.57079632679489678 -> xyz=-0.020822569739601552719 0.01393648576781737064 -0.016207791599192972187 rpy=-1.570796326794896558 0 1.57079632679489678

Commit message: added scrambled and unscrambled urdf

File: my-robot/robot.urdf (robot description, URDF)
Before this commit: robot onshape, 2 links, 1 joints
Links:
- link left_leg: mass 0.41395129653808809822 -> 0.4139512965380884868
- link right_leg: mass 0.39597688179033818656 -> 0.39597688179033829758
Joints:
- joint hip: limit effort=1 velocity=20 -> lower=-1.570796326794896558 upper=1.570796326794896558 effort=1 velocity=20; origin xyz=-0.020822569739601552719 0.01393648576781737064 -0.016207791599192972187 rpy=-1.570796326794896558 0 1.57079632679489678 -> xyz=-0.020822569739601518024 0.013936485767817355028 -0.016207791599193055454 rpy=-1.570796326794896558 -0 1.570796326794896558
