Commit message: duplo urdf

File: my-robot-fixed-scrambled/robot.urdf (robot description, URDF)
Before this commit: robot onshape, 10 links, 9 joints
Links:
- link left_leg: geometry collision mesh filename=package:///left_foot.stl; collision mesh filename=package:///left_leg.stl
- link left_leg_1: geometry visual mesh filename=package:///right_arm.stl
- link left_leg_2: geometry visual mesh filename=package:///right_battery.stl
- link left_leg_3: geometry visual mesh filename=package:///left_foot.stl
- link left_leg_4: geometry visual mesh filename=package:///left_leg.stl
- link right_leg: geometry collision mesh filename=package:///left_arm.stl; collision mesh filename=package:///right_battery.stl
- link right_leg_1: geometry visual mesh filename=package:///left_arm.stl
- link right_leg_2: mass None -> 1e-9; geometry visual mesh filename=package:///right_foot.stl
- link right_leg_3: geometry visual mesh filename=package:///right_leg.stl
- link right_leg_4: geometry visual mesh filename=package:///right_battery.stl
