Commit message: duplo ball feet import

File: zippy/robot.urdf (robot description, URDF)
Before this commit: robot onshape, 2 links, 1 joints
Joints:
- joint hip: limit lower=-0.34906585039886589561 upper=0.34906585039886589561 effort=1 velocity=20 -> lower=-0.34906585039886589561 upper=0.34906585039886589561
